File: Standard/snesypbpr-enhanced.kicad_sch (KiCad schematic)
At the start: 15 parts, among them J1 Pr In, J2 Pb In, J3 +5V, J4 GND, J5 Pr Out, J6 Pb Out, Q1 S8050/SS8050

Commit message: 2.0
Parts:
- removed R3, R4: 20R, Resistor_THT:R_Axial_DIN0204_L3.6mm_D1.6mm_P5.08mm_Horizontal, symbol Device:R_Small_US
- removed RV1: 0-100R, Potentiometer_SMD:Potentiometer_Bourns_TC33X_Vertical, symbol Device:R_Potentiometer_Trim_US
- added D2: 1N4148, Diode_THT:D_DO-35_SOD27_P7.62mm_Horizontal, symbol Diode:1N4148
- added Q2: S8050/SS8050, Package_TO_SOT_THT:TO-92_Inline_Wide, symbol Transistor_BJT:S8050
- C1, C2: value 220uF 35V -> 220uF 6.3V; footprint Capacitor_THT:CP_Radial_D8.0mm_P3.50mm -> Capacitor_THT:CP_Radial_D6.3mm_P2.50mm
- Q1: footprint Package_TO_SOT_THT:TO-92_Inline -> Package_TO_SOT_THT:TO-92_Inline_Wide
- R1, R2: value 20R -> 75R; footprint Resistor_THT:R_Axial_DIN0204_L3.6mm_D1.6mm_P5.08mm_Horizontal -> Resistor_THT:R_Axial_DIN0207_L6.3mm_D2.5mm_P7.62mm_Horizontal
Connections:
- net +5V: now also Q2.3 (C)
- net GND: now also R1.2, R2.2
- net at J6.1 (Pin_1): now also C2.2
- net at R2.1: now also C2.1, Q2.1 (E)
- net at J2.1 (Pin_1): now also D2.2 (A); no longer C2.1
- new net: D2.1 (K), Q2.2 (B)
- no-connect marks 1 -> 0
Other:
- moved on the sheet: J2, J3, J4
